Commit message: Trying to position mode

File: epos_hardware/launch/example.urdf (robot description, URDF)
Before this commit: robot example, 2 links, 1 joints
Joints:
- joint test_joint: limit (none) -> lower=0.01 upper=3.14159 effort=30.0 velocity=1.0

Commit message: new file:   epos_hardware/90-ftd2xx.rules 	new file:   epos_hardware/CHANGELOG.rst 	new file:   epos_hardware/CMakeLists.txt.user 	new file:   epos_hardware/epos_hardware.config 	new file:   epos_hardware/epos_hardware.creator 	new file:   epos_hardware/epos_hardware.creator.user 	new file:   epos_hardware/epos_hardware.files 	new file:   epos_hardware/epos_hardware.includes 	new file:   epos_hardware/install_udev_rules 	modified:   epos_hardware/launch/example.launch 	modified:   epos_hardware/launch/example.urdf 	modified:   epos_hardware/launch/example.yaml 	modified:   epos_hardware/src/nodes/epos_hardware_node.cpp 	modified:   epos_hardware/src/util/epos.cpp 	modified:   epos_hardware/src/util/epos_hardware.cpp 	modified:   epos_hardware/src/util/epos_manager.cpp

File: epos_hardware/launch/example.urdf (robot description, URDF)
Before this commit: robot example, 2 links, 1 joints
Links:
- added link link3, mass 1
- added link link4, mass 1
Joints:
- added joint test_joint3: type revolute, parent link3, child link4, limit lower=-10000.0 upper=10000.0 effort=3.0 velocity=10.0
- joint test_joint: limit lower=0.01 upper=3.14159 effort=30.0 velocity=1.0 -> lower=-10000.0 upper=10000.0 effort=3.0 velocity=10.0
